File: kicad_prj/MainBoard/cncc_v1.sch (KiCad schematic (older format))
At the start: 0 parts

Commit message: Corrected Conflicts
Capstone folder cleaned up
Changed lines of the file:
@@
 EESchema Schematic File Version 2
+LIBS:cncc_v1-rescue
 LIBS:power
 LIBS:device
@@
 $EndDescr
 $Sheet
-S 9150 1350 900  700
-U 56526EA5
-F0 "StepperDriverX" 60
-F1 "stp_drv.sch" 60
-F2 "VM" U R 10050 1500 60
-F3 "GND" U R 10050 1600 60
-F4 "STEP" I L 9150 1400 60
-F5 "DIR" I L 9150 1500 60
-F6 "EN" I L 9150 1600 60
-F7 "~SLEEP" I L 9150 1700 60
-F8 "VREF" I L 9150 2000 60
-F9 "~FAULT" O L 9150 1850 60
-$EndSheet
-$Sheet
-S 9150 2250 900  700
-U 5653D417
-F0 "StepperDriverY" 60
-F1 "stp_drv.sch" 60
-F2 "VM" U R 10050 2400 60
-F3 "GND" U R 10050 2500 60
-F4 "STEP" I L 9150 2300 60
-F5 "DIR" I L 9150 2400 60
-F6 "EN" I L 9150 2500 60
-F7 "~SLEEP" I L 9150 2600 60
-F8 "VREF" I L 9150 2900 60
-F9 "~FAULT" O L 9150 2750 60
-$EndSheet
-$Sheet
-S 9150 3150 900  700
-U 56542384
-F0 "StepperDriverZ" 60
-F1 "stp_drv.sch" 60
-F2 "VM" U R 10050 3300 60
-F3 "GND" U R 10050 3400 60
-F4 "STEP" I L 9150 3200 60
-F5 "DIR" I L 9150 3300 60
-F6 "EN" I L 9150 3400 60
-F7 "~SLEEP" I L 9150 3500 60
-F8 "VREF" I L 9150 3800 60
-F9 "~FAULT" O L 9150 3650 60
-$EndSheet
-$Sheet
-S 9150 4050 900  700
-U 5654C1EE
-F0 "StepperDriverA" 60
-F1 "stp_drv.sch" 60
-F2 "VM" U R 10050 4200 60
-F3 "GND" U R 10050 4300 60
-F4 "STEP" I L 9150 4100 60
-F5 "DIR" I L 9150 4200 60
-F6 "EN" I L 9150 4300 60
-F7 "~SLEEP" I L 9150 4400 60
-F8 "VREF" I L 9150 4700 60
-F9 "~FAULT" O L 9150 4550 60
-$EndSheet
-$Sheet
 S 6500 3500 900  750
 U 5653A94A
@@
 CH[0..3]
 $Sheet
-S 1750 1100 1550 3200
+S 1250 3300 1550 3200
 U 566CD168
 F0 "MCU_GPIO" 60
@@
 $EndSheet
 $Sheet
-S 1800 4700 1500 1750
+S 1300 1050 1500 1750
 U 566DECB3
 F0 "MCU_MAIN" 60
