File: kicad_prj/MainBoard/mcu_gpio.sch (KiCad schematic (older format))
At the start: 1 part

Commit message: Corrected Conflicts
Capstone folder cleaned up
Parts:
- U?: symbol TM4C1294NCPDT -> TM4C1294NCPDT-RESCUE-cncc_v1
Changed lines of the file:
@@
 EESchema Schematic File Version 2
+LIBS:cncc_v1-rescue
 LIBS:power
 LIBS:device
@@
 $EndDescr
 $Comp
-L TM4C1294NCPDT U?
+L TM4C1294NCPDT-RESCUE-cncc_v1 U?
 U 1 1 566CD626
 P 5450 3650
