File: kicad_prj/MainBoard/pow_in.sch (KiCad schematic (older format))
At the start: 35 parts

Commit message: Corrected Conflicts
Capstone folder cleaned up
Other:
- note removed: "NOTE: CORRECT PART SYMBOL"
Changed lines of the file:
@@
 EESchema Schematic File Version 2
+LIBS:cncc_v1-rescue
 LIBS:power
 LIBS:device
@@
 Text HLabel 9650 2650 2    60   UnSpc ~ 0
 +VDD_LP
-Text Notes 6350 4700 0    60   ~ 0
-NOTE: CORRECT PART SYMBOL
 $EndSCHEMATC
